File: Main/minisumo.kicad_sch (KiCad schematic)
At the start: 55 parts, among them J10 SDER, J11 PDER, J2 M_DER, J3 Conn_01x04_Pin, J4 M_IZ, J7 SIZQ, J8 SFRE, J9 PIZQ, SW1 SW_Push, SW2 SW_DIP_x02, SW3 SW_Push, SW4 SW_Push, SW6 SW_Nidec_CAS-120A1, U2 AMS1117-3.3, U3 TA6586, U4 ESP-WROOM-32, U5 TA6586, U6 Mini360

Commit message: actualizado
Parts:
- J10, J11, J7, J8, J9: footprint Connector_JST:JST_EH_B3B-EH-A_1x03_P2.50mm_Vertical -> Connector_JST:JST_XH_B3B-XH-A_1x03_P2.50mm_Vertical
Other:
- note added: "Connector_JST:JST_XH_B3B-XH-A_1x03_P2.50mm_Vertical"
Changed lines of the file:
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@@
 		)
 	)
+	(text "Connector_JST:JST_XH_B3B-XH-A_1x03_P2.50mm_Vertical\n"
+		(exclude_from_sim no)
+		(at 117.348 14.224 0)
+		(effects
+			(font
+				(size 1.27 1.27)
+			)
+		)
+	)
 	(text "DRIVERS Y BAT\n"
 		(exclude_from_sim no)
@@
 			"RABIAHgAQgAwAHUAWgB3AFYAYwBCAGkAagBnAFgAYwBCACsANABBAGYAdQBEAHUAeAAvAFoAZwBY"
 			"AHcAUQBlAEIAegB3AEEAcgBnAEIAdQBBAHMAbwBBAGEAOABEAHYAagB3AGMAVgBjADQAdwA0AE8A"
-			"aABNAA=="
+			"aABNAAAAAAAAAAAAAAAAAAAAAAAAAAAAAAAAAAAAAAAAAAAAAAAAAAAAAAAAAAAAAAAAAAAAAAAA"
+			"AAAAAAAAAAAAAAAAAAAAAAAAAAAAAAAAAAAAAAAAAAAAAAAAAAAAAAAAAAAAAAAAAAAAAAAAAAAA"
+			"AAAAAAAAAAAAAAAAAAAAAAAAAAAAAAAAAAAAAAAAAAAAAAAAAAAAAAAAAAAAAAAAAAAAAAAAAAAA"
+			"AAAAAAAAAAAAAAAAAAAAAAAAAAAAAAAAAAAAAAAAAAAAAAAAAAAAAAAAAAAAAAAAAAAAAAAAAAAA"
+			"AAAAAAAAAAAAAAAAAAAAAAAAAAAAAAAAAAAAAAAAAAAAAAAAAAAAAAAAAAAAAAAAAAAAAAAAAAAA"
+			"AAAAAAAAAAAAAAAAAAAAAAAAAAAAAAAAAAAAAAAAAAAAAAAAAAAAAAAAAAAAAAAAAAAAAAAAAAAA"
+			"AAAAAAAAAAAAAAAAAAAAAAAAAAAAAAAAAAAAAAAAAAAAAAAAAAAAAAAAAAAAAAAAAAAAAAAAAAAA"
+			"AAAAAAAAAAAAAAAAAAAAAAAAAAAAAAAAAAAAAAAAAAAAAAAAAAAAAAAAAAAAAAAAAAAAAAAAAAAA"
+			"AABSAFoAOABnAHYAdgBMAGwATAA5ACsAOQBlADkAZgBWAHoAMwAzAEIANwBUACsANQA5AGQAdgBm"
+			"AC8AZwA2AEEAcwA4ADcAWQA5AGgAZAAvADgAMgBrAGgAeABKAHEAMQA2ADgANAAvAC8ANwB4AGIA"
+			"YgAvADMASgA4AGIANgBiAEYAKwBiAG4ALwA0AEYAOQB4AHgAMQAzAHUASABHAGUAUwBCAFMAWgB6"
+			"AFoATwBDAEwASQBTAFEAcgBpAFIAYwBsAEEAcQBuAEQAawB0AHcAawBvADgARQBPAHUAcgBvAE0A"
+			"cwBBADAAQwBXAFIAMABZAFgAWABoAEYAdQAzAFcARgBlADkATABVADIAaABkAG0ARQBJAEkAdwBV"
+			"AHgASwBTAFcATgBLAEgALwBNAEIATQAxAFMAVQBRAHIAUgBNAGcARABQAGUAcABtAFAAcwBYADkA"
+			"ZwBCAGIAWQBNAFMAZgBpAEgARQBBAGsAWABhAEkAWABZAHEAVwAyAGIARgBMAEsAVQBVAFYASABv"
+			"AFQATwBaAHoAVQBsAFIAZwA3AHcASgBSAEsAZgBMAEoAdwBRAEgAQwBtAGkAegB6AFAAMQA2AHgA"
+			"ZQByAFQAegBQADgANwB4AHUAdAA5AHUAYQBhADIAWgBaAE8AZwBCAHQAOAB6AHgAMwBxAHEAQgA1"
+			"AG4AcgBzAGYAcgB0AGYAcgBTAGkAbQAzAEQAbgBTADYAcQBrAEoASwBFAGkATABQADgAegB6AFAA"
+			"SABiAA=="
 		)
 	)
@@
 			)
 		)
-		(property "Footprint" "Connector_JST:JST_EH_B3B-EH-A_1x03_P2.50mm_Vertical"
+		(property "Footprint" "Connector_JST:JST_XH_B3B-XH-A_1x03_P2.50mm_Vertical"
 			(at 83.82 66.675 0)
 			(effects
@@
 			)
 		)
-		(property "Footprint" "Connector_JST:JST_EH_B3B-EH-A_1x03_P2.50mm_Vertical"
+		(property "Footprint" "Connector_JST:JST_XH_B3B-XH-A_1x03_P2.50mm_Vertical"
 			(at 102.87 22.86 0)
 			(effects
@@
 			)
 		)
-		(property "Footprint" "Connector_JST:JST_EH_B3B-EH-A_1x03_P2.50mm_Vertical"
+		(property "Footprint" "Connector_JST:JST_XH_B3B-XH-A_1x03_P2.50mm_Vertical"
 			(at 85.725 22.86 0)
 			(effects
@@
 			)
 		)
-		(property "Footprint" "Connector_JST:JST_EH_B3B-EH-A_1x03_P2.50mm_Vertical"
+		(property "Footprint" "Connector_JST:JST_XH_B3B-XH-A_1x03_P2.50mm_Vertical"
 			(at 85.09 45.085 0)
 			(effects
@@
 			)
 		)
-		(property "Footprint" "Connector_JST:JST_EH_B3B-EH-A_1x03_P2.50mm_Vertical"
+		(property "Footprint" "Connector_JST:JST_XH_B3B-XH-A_1x03_P2.50mm_Vertical"
 			(at 104.14 66.675 0)
 			(effects

Commit message: actual
Parts:
- C7: renamed from C100nF3; value C -> 100nF
- C8: renamed from C100nF1; value C -> 100nF
- D8: value MODO1 -> M1
- D9: value MODO2 -> M2
- J3: value Conn_01x04_Pin -> USB
- R1: renamed from R330; value R -> 330
- R10: renamed from R9; value R 1OK -> 10K
- R11: renamed from R10K2; value R -> 10K
- R12: renamed from R10K1; value R -> 10K
- R4: renamed from R1; value 470 Azul -> 330
- R5: renamed from R2; value 220 Rojo -> 330
- R6: renamed from R8; value R 330 -> 330
- R7: renamed from R10; value R 330 -> 330
- SW1: value SW_Push -> ACT
- SW3: value SW_Push -> EN
- SW4: value SW_Push -> BOOT
- renumbered C13 to C1, C9 to C10, C10 to C11, C17 to C2, C14 to C3, C15 to C4, C8 to C6, C11 to C9, C16 to CE1, C12 to CE2, C6 to CE3, C7 to CE4, R4 to R2, R11 to R8, R12 to R9
Connections:
- net GND: now also R8.2, R9.2; no longer SW6.1 (C)
- net at R6.2: now also D8.2 (A); no longer R8.1
- net at R7.2: now also D9.2 (A); no longer R9.1
- net AUTO renamed M1
- net M1: now also R8.1
- net BAT renamed VCC
- net RC renamed M2
- net M2: now also R9.1
- no-connect marks 17 -> 18
Other:
- note added: "BAT 11.1V 650MAH"
- note added: "CE1-2=470uF CE3-4=100uF C=100nF R1-7=330 R8-11=10K ______________"
- note removed: "CAP 470uF 25V CAP 100nF 25V"
- note removed: "Connector_JST:JST_XH_B3B-XH-A_1x03_P2.50mm_Vertical"
- moved on the sheet: D8, H1, H2, R6, R7, R8, R9, SW2
