File: Main/minisumo.kicad_sch (KiCad schematic)
At the start: 56 parts, among them J10 SDER, J11 PDER, J2 M_IZ, J3 USB, J4 M_DER, J7 SIZQ, J8 SFRE, J9 PIZQ, SW1 ACT, SW2 SW_DIP_x02, SW3 EN, SW4 BOOT, SW6 SW_Nidec_CAS-120A1, U2 AMS1117-3.3, U3 TA6586, U4 ESP-WROOM-32, U5 TA6586, U6 Mini360

Commit message: .
Parts:
- removed D1: Azul, LED_SMD:LED_0805_2012Metric_Pad1.15x1.40mm_HandSolder, symbol Device:LED
- removed D2: Rojo, LED_SMD:LED_0805_2012Metric_Pad1.15x1.40mm_HandSolder, symbol Device:LED
- removed R4: 330, LED_SMD:LED_0805_2012Metric_Pad1.15x1.40mm_HandSolder, symbol Device:R
- removed R5: 330, Resistor_SMD:R_0805_2012Metric_Pad1.20x1.40mm_HandSolder, symbol Device:R
- J2: value M_IZ -> M_DER
- J4: value M_DER -> M_IZ
Connections:
- net VCC: no longer C1.2, C3.2, U3.VCC, U5.VCC
- net +BATT: now reaches BAT1.2 (Pin_2), SW6.2 (B)
- net +BATT: now also C1.2, C3.2, U3.VCC, U5.VCC

Commit message: .
Parts:
- renumbered R12 to R10, R6 to R4, R7 to R5, R8 to R6, R9 to R7, R10 to R8, R11 to R9
Other:
- note added: "CE2=100uF CE3-4=1uF C=100nF R1-5=330 R6-10=10K ______________"
- note removed: "CE2=100uF CE3-4=1uF C=100nF R1-7=330 R8-11=10K ______________"
Changed lines of the file:
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@@
 		)
 	)
-	(text "CE2=100uF\nCE3-4=1uF\nC=100nF\nR1-7=330\nR8-11=10K\n______________\n"
+	(text "CE2=100uF\nCE3-4=1uF\nC=100nF\nR1-5=330\nR6-10=10K\n______________\n"
 		(exclude_from_sim no)
 		(at 150.876 161.036 0)
@@
 			"NwB6AHQATwBsAHUAagB4AEoAeABFAHAATQA3AFAAQgB5AFAATABqAEEAYwAxAHUAOQBjAFEAdgBE"
 			"AEYAUQBzAFcAbQBTAEoARgBYADEARgBKAGkAcABrADUASwAyAEMAVgBkAEkASwBUAGwASABSAE8A"
-			"UwBkAA=="
+			"UwBkAEsAVABsAEgAUgBPAFMAZABWADkAVQBrAGEAYgBRADIAQQBxAEQAUQBzAGkAaQBKAG4AVwBx"
+			"AE8AdABTAEcAMgBaAEMAMQBtAGQAagBGAEYAVgBUAFUAcQBxAE8AcwA5AEYAYQAxAGoAYgBlAHAA"
+			"SQBBAE0AUgBrADkARwBKAFIARgB1AGgATQBhAEUAMwBoAHEAMQByAFYAdABVAFUARABwAFoAUgBp"
+			"AFQARQBRAHcAOQBoAFEARQBFAFUAawB4AHgAUgBSAEgAWQB6AFcAbABaAEcAdQBGAG0AWgBJAGsA"
+			"NQAvAHkAZwBQADEAUAAwAFMAMgBiAFQANQBLADIATABlAFQAcwBiAEIATwB0AEcAWQA0AGUANQBY"
+			"AFUALwBSAEMAbwAxAGIAMQA4AGkAbQBhAFUAUQBqAEUAUQAwAEcAdgBaAGEAMQBBAHoARwBEAHEA"
+			"YQB1AEMATgArAEsAcQBpAFgAVwBzAG8AMgBNAHUAZwBtAFAAbQBFAEQAdwBUAEsAOABFAFoAbwBV"
+			"AFgAYwBiAHEAMwBtAGMAMgBwAFUAbwA0AFUARwAxAFYAVwBkAGsAcQByAGsASwAwADUARQAzAHIA"
+			"dgB1AFcAcQB2AEcASgBxAFkAawB1AGYASABrAHYAQwBkADIAegByAEcAagBwAHEAbQA5ADgAOAB5"
+			"AGMASgBNAFUAWQBxADYAcABLAGsAawBTADAAcQBaAHUAVQB4AEwAUwBOADEATQBKAEkALwAyADYA"
+			"SgBhAGEAVgB0AEwATQBVAFkAdgBmAGMAeAB4AHEAbwBlAHAAWgBpAEkAcQBQAFUAQQB6AGEAagBx"
+			"AGkAdABEAFcAZwBMAGQAQwA0AEsAcQBxAHoAUQArAGgATABFAHYAcgB6AEsAYgBKAHkAbABaAFYA"
+			"VwBWAHgAYwBhAEcASQBUAG0AMgBRAHMAdABpAFMANwBwADgAaAA0AGYAdQA4ADkAawB4AFAAUgAw"
+			"AFcAaQBjADcAeQBNAGkAUwBSAHAAOABVAFYAVwAxAEQAZQBTAHEAcgBwAGUAVwBsADYAMwBIAHkA"
+			"cgBJAHMAUwArAE4AcQAxAC8AWABnADEAcgBiAHUAVABnAEcAUgBZADgAZQBCAFQAUQB3AGIAUQBw"
+			"AEQAMQBNAG4AawBDAEUARgBOAGMAWABLADYAdwB0AEwAeQA4AE0AdgBUAE8AOQAvAHQAbABDAEEA"
+			"SABNAGcATgBqAFEAUwB5AHIATwBlADQARgBLAFQASwBKAFMATgAzAFYAcwBJAHQAbwBFAHAAMABi"
+			"AFMAYQBHADEAawBOADAAcwBlAFMASwBKAEoAawBoAHUATgA4ADUAMgBlAHgAWgAzADIANABLAEQA"
+			"ZwBjAA=="
 		)
 	)
@@
 		(on_board yes)
 		(dnp no)
-		(property "Reference" "R8"
+		(property "Reference" "R6"
 			(at 180.975 19.177 90)
 			(effects
@@
 			(project "minisumo"
 				(path "/abeb3225-9534-4616-a1ab-54bb3ef1c7bc"
-					(reference "R8")
+					(reference "R6")
 					(unit 1)
 				)
@@
 		(on_board yes)
 		(dnp no)
-		(property "Reference" "R7"
+		(property "Reference" "R5"
 			(at 180.848 25.4 90)
 			(effects
@@
 			(project "minisumo"
 				(path "/abeb3225-9534-4616-a1ab-54bb3ef1c7bc"
-					(reference "R7")
+					(reference "R5")
 					(unit 1)
 				)
@@
 		(on_board yes)
 		(dnp no)
-		(property "Reference" "R6"
+		(property "Reference" "R4"
 			(at 180.975 22.987 90)
 			(effects
@@
 			(project "minisumo"
 				(path "/abeb3225-9534-4616-a1ab-54bb3ef1c7bc"
-					(reference "R6")
+					(reference "R4")
 					(unit 1)
 				)
@@
 		(on_board yes)
 		(dnp no)
-		(property "Reference" "R9"
+		(property "Reference" "R7"
 			(at 180.975 29.972 90)
 			(effects
@@
 			(project "minisumo"
 				(path "/abeb3225-9534-4616-a1ab-54bb3ef1c7bc"
-					(reference "R9")
+					(reference "R7")
 					(unit 1)
 				)
@@
 		(on_board yes)
 		(dnp no)
-		(property "Reference" "R12"
+		(property "Reference" "R10"
 			(at 109.982 158.242 90)
 			(effects
@@
 			(project "minisumo"
 				(path "/abeb3225-9534-4616-a1ab-54bb3ef1c7bc"
-					(reference "R12")
+					(reference "R10")
 					(unit 1)
 				)
@@
 		(on_board yes)
 		(dnp no)
-		(property "Reference" "R10"
+		(property "Reference" "R8"
 			(at 129.54 46.99 90)
 			(effects
@@
 			(project "minisumo"
 				(path "/abeb3225-9534-4616-a1ab-54bb3ef1c7bc"
-					(reference "R10")
+					(reference "R8")
 					(unit 1)
 				)
@@
 		(on_board yes)
 		(dnp no)
-		(property "Reference" "R11"
+		(property "Reference" "R9"
 			(at 62.992 158.75 90)
 			(effects
@@
 			(project "minisumo"
 				(path "/abeb3225-9534-4616-a1ab-54bb3ef1c7bc"
-					(reference "R11")
+					(reference "R9")
 					(unit 1)
 				)
