File: Main/minisumo.kicad_pcb (KiCad board)
At the start: 2 copper layers, 86.5 x 36.5 mm, 55 parts, among them J10 SDER, J11 PDER, J2 M_DER, J3 Conn_01x04_Pin, J4 M_IZ, J7 SIZQ, J8 SFRE, J9 PIZQ, SW1 SW_Push, SW2 SW_DIP_x02, SW3 SW_Push, SW4 SW_Push, SW6 SW_Nidec_CAS-120A1, U2 AMS1117-3.3, U3 TA6586, U4 ESP-WROOM-32, U5 TA6586, U6 Mini360

Commit message: actualizado
Parts:
- added G***: LOGO, er:111, F.Cu at (205.7, 74.5)
- J10, J11, J7, J8, J9: footprint Connector_JST:JST_EH_B3B-EH-A_1x03_P2.50mm_Vertical -> Connector_JST:JST_XH_B3B-XH-A_1x03_P2.50mm_Vertical
- moved J11 2.09 mm to (207.2, 60.5)
- moved J10 1.99 mm to (196.3, 60.5)
- moved J8 1.90 mm to (185.4, 60.5)
- moved J7 1.80 mm to (174.5, 60.5)
- moved J9 1.62 mm to (163.6, 60.5)
Routing:
- net GND: track 13.9 -> 11.0 mm
- net P_DER: track 49.0 -> 46.2 mm, vias 1 -> 3
- net F_DER: track 31.3 -> 28.7 mm
- net F_FRE: track 23.3 -> 20.7 mm
- net +3.3V: track 167.0 -> 165.0 mm
- net P_IZ: track 9.10 -> 7.42 mm, vias 0 -> 1
- net F_IZ: track 22.7 -> 21.1 mm
- net +5V: track 87.0 -> 87.9 mm
- net RXDO: track 26.6 -> 26.7 mm, vias 2 -> 0
Other:
- board text added: "CE 1-2 :470uF CE 3-4 :100uF C 1-11 :100nF R 1-7 :330 R 8-12 :10K"

Commit message: actual
Parts:
- C7: renamed from C100nF3; value C -> 100nF
- C8: renamed from C100nF1; value C -> 100nF
- D8: value MODO1 -> M1
- D9: value MODO2 -> M2
- J3: value Conn_01x04_Pin -> USB
- R1: renamed from R330; value R -> 330
- R10: renamed from R9; value R 1OK -> 10K
- R11: renamed from R10K2; value R -> 10K
- R12: renamed from R10K1; value R -> 10K
- R4: renamed from R1; value 470 Azul -> 330
- R5: renamed from R2; value 220 Rojo -> 330
- R6: renamed from R8; value R 330 -> 330
- R7: renamed from R10; value R 330 -> 330
- SW1: value SW_Push -> ACT
- SW3: value SW_Push -> EN
- SW4: value SW_Push -> BOOT
- moved R9 2.13 mm to (196.5, 65.0)
- moved D9 2.10 mm to (198.6, 65.0)
- moved D8 2.05 mm to (191.9, 65.0)
- moved R8 2.03 mm to (193.9, 65.0)
- renumbered C13 to C1, C9 to C10, C10 to C11, C17 to C2, C14 to C3, C15 to C4, C8 to C6, C11 to C9, C16 to CE1, C12 to CE2, C6 to CE3, C7 to CE4, R4 to R2, R11 to R8, R12 to R9
Connections:
- net BAT renamed VCC
- R6 pad 1: AUTO -> M1
- R6 pad 2: Net-(R11-Pad1) -> Net-(D8-A)
- R7 pad 1: RC -> M2
- R7 pad 2: Net-(R10-Pad2) -> Net-(D9-A)
- R8 pad 1: Net-(R11-Pad1) -> M1
- R8 pad 2: Net-(D8-A) -> GND
- R9 pad 1: Net-(R10-Pad2) -> M2
- R9 pad 2: Net-(D9-A) -> GND
- SW2 pad 3: RC -> M2
- SW2 pad 4: AUTO -> M1
- SW6 pad 1: GND -> unconnected-(SW6-C-Pad1)
- U4 pad 13: AUTO -> M1
- U4 pad 26: RC -> M2
Routing:
- net M1: track 0.00 -> 35.5 mm, vias 0 -> 2
- net AUTO: track 33.0 -> 0.00 mm, vias 2 -> 0
- net M2: track 0.00 -> 31.6 mm, vias 0 -> 2
- net RC: track 29.1 -> 0.00 mm, vias 2 -> 0
- net Net-(R11-Pad1): track 9.32 -> 0.00 mm, vias 1 -> 0
- net Net-(R10-Pad2): track 9.31 -> 0.00 mm, vias 1 -> 0
- net GND: track 11.0 -> 3.17 mm
- net Net-(D8-A): track 2.88 -> 9.30 mm, vias 0 -> 1
- net Net-(D9-A): track 2.93 -> 9.28 mm, vias 0 -> 1
- net +3.3V: track 165.0 -> 170.3 mm
- net RXDO: track 26.7 -> 27.8 mm
- net WS3: track 21.1 -> 21.9 mm
Other:
- board size 86.5 x 36.5 mm -> 86.5 x 36.6 mm
- board text added: "CE1-2=470uF CE3-4=100uF C=100nF R1-7=330 R8-11=10K"
- board text removed: "CE 1-2 :470uF CE 3-4 :100uF C 1-11 :100nF R 1-7 :330 R 8-12 :10K"

Commit message: vaquin
Parts:
- removed CE1: 470uF, Capacitor_Tantalum_SMD:CP_EIA-7343-43_Kemet-X
- added H3: MountingHole, MountingHole:MountingHole_2.2mm_M2_ISO7380, F.Cu at (151.3, 90.4)
- added H4: MountingHole, MountingHole:MountingHole_2.2mm_M2_ISO7380, F.Cu at (226.2, 90.4)
- CE2: value 470uF -> 100uF; footprint Capacitor_Tantalum_SMD:CP_EIA-7343-43_Kemet-X -> Capacitor_Tantalum_SMD:CP_EIA-7343-20_Kemet-V_HandSolder; moved to B.Cu
- CE3: value 100uf -> 1uf; footprint Capacitor_THT:CP_Radial_D8.0mm_P3.50mm -> Capacitor_SMD:C_0805_2012Metric_Pad1.18x1.45mm_HandSolder
- CE4: value 100uF -> 1uF; footprint Capacitor_THT:CP_Radial_D8.0mm_P3.50mm -> Capacitor_SMD:C_0805_2012Metric_Pad1.18x1.45mm_HandSolder
- moved CE3 21.1 mm to (206.4, 65.3)
- moved CE2 14.6 mm to (214.2, 73.0)
- moved BAT1 13.4 mm to (210.2, 88.2)
- moved SW6 13.2 mm to (199.9, 88.2)
- moved J4 13.0 mm to (219.2, 88.0)
- moved CE4 11.9 mm to (202.1, 77.7)
- moved C5 11.5 mm to (206.4, 67.3)
- moved H2 6.50 mm to (226.2, 58.9)
- moved R3 6.19 mm to (195.6, 86.6)
- moved LED2 6.19 mm to (178.5, 88.3)
- moved LED3 6.19 mm to (189.9, 88.3)
- moved C8 6.19 mm to (184.2, 89.1)
- moved C9 6.19 mm to (195.6, 89.1)
- moved R2 6.19 mm to (184.2, 86.6)
- moved LED1 6.19 mm to (167.3, 88.3)
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Connections:
- CE2 pad 1: GND -> VCC
- CE2 pad 2: VCC -> GND
Routing:
- net Net-(J2-Pin_2): track 120.0 -> 102.7 mm, vias 0 -> 1
- net Net-(J2-Pin_1): track 114.6 -> 99.6 mm
- net VCC: track 50.9 -> 40.1 mm
- net Net-(J4-Pin_2): track 27.9 -> 18.2 mm
- net +3.3V: track 170.3 -> 161.8 mm, vias 2 -> 5
- net Net-(J4-Pin_1): track 26.0 -> 19.2 mm
- net WS3: track 21.9 -> 28.6 mm
- net WS2: track 11.8 -> 18.5 mm
- net +5V: track 87.9 -> 83.5 mm, vias 3 -> 1
- net BI_DER: track 60.1 -> 56.2 mm
- net FI_IZ: track 58.7 -> 62.5 mm, vias 0 -> 1
- net WS1: track 5.06 -> 8.47 mm
- net BI_IZQ: track 54.7 -> 51.7 mm
- net Net-(LED1-DIN): track 3.30 -> 2.10 mm
- net Net-(BAT1-Pin_2): track 6.17 -> 5.38 mm
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Other:
- board size 86.5 x 36.6 mm -> 80 x 36.6 mm
- board text added: "CE2=100uF CE3-4=1uF C=100nF R1-7=330 R8-11=10K"
- board text removed: "CE1-2=470uF CE3-4=100uF C=100nF R1-7=330 R8-11=10K"

Commit message: fack
Parts:
- moved R6 0.15 mm to (193.9, 73.0)
- moved C1 0.07 mm to (219.0, 69.9)
- moved C3 0.07 mm to (219.0, 80.5)
- moved C4 0.07 mm to (222.0, 77.6)
Routing:
- net VCC: track 40.1 -> 2.78 mm
- net P_IZ: track 7.42 -> 13.8 mm
- net GND: track 3.07 -> 0.17 mm
- net Net-(J2-Pin_2): track 102.7 -> 104.4 mm
- net P_DER: track 46.2 -> 47.5 mm, vias 3 -> 2
- net FI_IZ: track 62.5 -> 63.1 mm
- net Net-(J2-Pin_1): track 99.6 -> 100.2 mm
- net Net-(J4-Pin_1): track 19.2 -> 18.7 mm
- net EN: track 28.9 -> 28.3 mm
- added copper zone on B.Cu, net VCC
- added copper zone on F.Cu, net VCC
Other:
- copper layers 2 -> 4

Commit message: .
Parts:
- J2: value M_DER -> M_IZ
- J4: value M_IZ -> M_DER
- moved C1 0.33 mm to (219.0, 70.2)
Routing:
- net +3.3V: track 162.0 -> 99.2 mm
- net Net-(J2-Pin_2): track 104.4 -> 98.7 mm
- net Net-(J2-Pin_1): track 100.2 -> 95.1 mm
- net Net-(J4-Pin_2): track 18.4 -> 13.3 mm
- net Net-(J4-Pin_1): track 18.7 -> 13.8 mm
- added copper zone on B.Cu, net +3.3V
- added copper zone on F.Cu, net +3.3V
- added copper zone on F.Cu, net Net-(J2-Pin_1)
- added copper zone on F.Cu, net Net-(J2-Pin_2)
- added copper zone on F.Cu, net Net-(J4-Pin_1)
- added copper zone on F.Cu, net Net-(J4-Pin_2)
Other:
- board text added: "PDER"
- board text added: "PIZQ"
- board text added: "SDER"
- board text added: "SFRE"
- board text added: "SIZQ"

Commit message: .
Routing:
- net Net-(J2-Pin_1): track 95.1 -> 0.08 mm
- net Net-(J2-Pin_2): track 98.7 -> 6.96 mm
- net GND: track 0.17 -> 0.83 mm
- added copper zone on B.Cu, net Net-(J2-Pin_2)
Changed lines of the file:
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@@
+	)
+	(segment
+		(start 220.025 72.232)
+		(end 220.49 72.697)
+		(width 0.25)
+		(layer "F.Cu")
+		(net 1)
 	)
 	(segment
@@
 	)
 	(segment
-		(start 227.82 85.355)
-		(end 221.026 92.149)
-		(width 1)
-		(layer "F.Cu")
-		(net 15)
-	)
-	(segment
 		(start 223.105 67.525)
 		(end 223.05 67.47)
@@
 	)
 	(segment
-		(start 227.82 68.82)
-		(end 227.82 85.355)
+		(start 221.03 67.525)
+		(end 221.03 68.73)
 		(width 1)
 		(layer "F.Cu")
-		(net 15)
-	)
-	(segment
-		(start 223.105 67.525)
-		(end 223.13 67.5)
+		(net 16)
+	)
+	(segment
+		(start 221.65 69.35)
+		(end 226.53 69.35)
 		(width 1)
 		(layer "F.Cu")
-		(net 15)
-	)
-	(segment
-		(start 162.199 92.149)
-		(end 160.725 90.675)
-		(width 1)
-		(layer "F.Cu")
-		(net 15)
-	)
-	(segment
-		(start 226.5 67.5)
-		(end 227.82 68.82)
-		(width 1)
-		(layer "F.Cu")
-		(net 15)
-	)
-	(segment
-		(start 223.13 67.5)
-		(end 226.5 67.5)
-		(width 1)
-		(layer "F.Cu")
-		(net 15)
-	)
-	(segment
-		(start 160.725 90.675)
-		(end 160.725 87.975)
-		(width 1)
-		(layer "F.Cu")
-		(net 15)
-	)
-	(segment
-		(start 221.026 92.149)
-		(end 162.199 92.149)
-		(width 1)
-		(layer "F.Cu")
-		(net 15)
-	)
-	(segment
-		(start 226.53 69.35)
-		(end 222.1 69.35)
-		(width 1)
-		(layer "F.Cu")
 		(net 16)
 	)
 	(segment
-		(start 222.1 69.35)
-		(end 221.03 68.28)
-		(width 1)
-		(layer "F.Cu")
-		(net 16)
-	)
-	(segment
-		(start 221.03 68.28)
-		(end 221.03 68.13)
+		(start 221.03 68.73)
+		(end 221.65 69.35)
 		(width 1)
 		(layer "F.Cu")
@@
 		(drill 0.5)
 		(layers "F.Cu" "B.Cu")
-		(net 16)
-	)
-	(segment
-		(start 226.53 69.35)
-		(end 227.12 69.35)
-		(width 1)
-		(layer "B.Cu")
-		(net 16)
-	)
-	(segment
-		(start 159.774 92.149)
-		(end 158.225 90.6)
-		(width 1)
-		(layer "B.Cu")
-		(net 16)
-	)
-	(segment
-		(start 221.026 92.149)
-		(end 159.774 92.149)
-		(width 1)
-		(layer "B.Cu")
-		(net 16)
-	)
-	(segment
-		(start 227.12 69.35)
-		(end 227.82 70.05)
-		(width 1)
-		(layer "B.Cu")
-		(net 16)
-	)
-	(segment
-		(start 158.225 90.6)
-		(end 158.225 87.975)
-		(width 1)
-		(layer "B.Cu")
-		(net 16)
-	)
-	(segment
-		(start 227.82 70.05)
-		(end 227.82 85.355)
-		(width 1)
-		(layer "B.Cu")
-		(net 16)
-	)
-	(segment
-		(start 227.82 85.355)
-		(end 221.026 92.149)
-		(width 1)
-		(layer "B.Cu")
 		(net 16)
 	)
@@
 			(pts
 				(xy 222 74.25) (xy 226.5 74.25) (xy 226.5 76.75) (xy 224 76.75) (xy 224 78.75) (xy 222 78.75)
+			)
+		)
+	)
+	(zone
+		(net 15)
+		(net_name "Net-(J2-Pin_1)")
+		(layer "F.Cu")
+		(hatch edge 0.5)
+		(priority 9)
+		(connect_pads yes
+			(clearance 0.3)
+		)
+		(min_thickness 0.25)
+		(filled_areas_thickness no)
+		(fill yes
+			(thermal_gap 0.5)
+			(thermal_bridge_width 0.5)
+		)
+		(polygon
+			(pts
+				(xy 222 63.25) (xy 228.8 63.2) (xy 228.8 85.6) (xy 221.2 93) (xy 159.4 93) (xy 159.4 92.353855)
+				(xy 159.4 86.2) (xy 163.2 86.2) (xy 163.2 91.2) (xy 163.2 91.2) (xy 219.783765 90.602284) (xy 226.203769 84.596474)
+				(xy 226.4 68.5) (xy 222.070875 68.5)
 			)
 		)
@@
 		(polygon
 			(pts
-				(xy 216.5 63.25) (xy 221.75 63.25) (xy 221.76 68.5) (xy 220.25 68.5) (xy 220.25 66.776) (xy 216.5 66.776)
+				(xy 216.5 63.25) (xy 221.75 63.25) (xy 221.76 68.5) (xy 220.2 68.5) (xy 220.2 66.8) (xy 216.5 66.776)
 			)
 		)
@@
 			)
 		)
+	)
+	(zone
+		(net 16)
+		(net_name "Net-(J2-Pin_2)")
+		(layer "B.Cu")
+		(hatch edge 0.5)
+		(priority 10)
+		(connect_pads yes
+			(clearance 0.3)
+		)
+		(min_thickness 0.25)
+		(filled_areas_thickness no)
+		(fill yes
+			(thermal_gap 0.5)
+			(thermal_bridge_width 0.5)
+		)
+		(polygon
+			(pts
+				(xy 159.4 86.2) (xy 155.6 86.2) (xy 155.6 93) (xy 221.2 93) (xy 228.8 85.6) (xy 228.8 68.4) (xy 226 68.4)
+				(xy 226 84.6) (xy 219.8 90.8) (xy 159.4 90.8)
+			)
+		)

Commit message: .
Parts:
- removed D1: Azul, LED_SMD:LED_0805_2012Metric_Pad1.15x1.40mm_HandSolder
- removed D2: Rojo, LED_SMD:LED_0805_2012Metric_Pad1.15x1.40mm_HandSolder
- removed R4: 330, LED_SMD:LED_0805_2012Metric_Pad1.15x1.40mm_HandSolder
- removed R5: 330, Resistor_SMD:R_0805_2012Metric_Pad1.20x1.40mm_HandSolder
- C1, C2, C3, C4, C6: moved to B.Cu
- J2: value M_IZ -> M_DER
- J4: value M_DER -> M_IZ
- U3, U5: moved to F.Cu
- moved J2 55.3 mm to (216.0, 88.7)
- moved U3 30.1 mm to (212.2, 89.3), turned to -90 degrees
- moved SW6 28.4 mm to (220.2, 68.3)
- moved U5 25.8 mm to (201.7, 89.3), turned to -90 degrees
- moved C6 23.7 mm to (216.7, 70.1), turned to -90 degrees
- moved C4 18.2 mm to (204.3, 82.0)
- moved C3 17.6 mm to (201.5, 78.8)
- moved C2 16.1 mm to (214.8, 81.9)
- moved CE4 14.6 mm to (214.6, 70.1), turned to -90 degrees
- moved J4 13.7 mm to (205.5, 88.8)
- moved CE2 13.2 mm to (219.8, 61.1), turned to 0 degrees
- moved BAT1 13.1 mm to (223.0, 85.2), turned to 90 degrees
- moved C9 11.7 mm to (183.9, 88.0)
- moved R3 11.7 mm to (183.9, 85.5)
- moved LED3 11.5 mm to (178.5, 87.2)
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Connections:
- BAT1 pad 2: Net-(BAT1-Pin_2) -> +BATT
- C1 pad 2: VCC -> +BATT
- C3 pad 2: VCC -> +BATT
- SW6 pad 2: Net-(BAT1-Pin_2) -> +BATT
- U3 pad VCC: VCC -> +BATT
- U5 pad VCC: VCC -> +BATT
Routing:
- net +5V: track 83.1 -> 35.5 mm
- net BI_IZQ: track 51.8 -> 37.5 mm, vias 0 -> 1
- net BI_DER: track 56.4 -> 42.3 mm, vias 0 -> 1
- net Net-(J4-Pin_1): track 13.8 -> 0.00 mm
- net +3.3V: track 99.2 -> 85.7 mm, vias 5 -> 2
- net Net-(J4-Pin_2): track 13.3 -> 0.00 mm
- net WS3: track 28.6 -> 16.0 mm
- net WS2: track 18.4 -> 6.48 mm
- net FI_IZ: track 63.1 -> 53.3 mm, vias 1 -> 0
- net Net-(J2-Pin_2): track 6.96 -> 0.00 mm, vias 1 -> 0
- net Net-(BAT1-Pin_2): track 5.39 -> 0.00 mm
- net BI_IZ: track 59.1 -> 54.3 mm, vias 1 -> 0
- net Net-(D1-A): track 3.21 -> 0.00 mm, vias 1 -> 0
- net Net-(D2-A): track 3.13 -> 0.00 mm, vias 1 -> 0
- net VCC: track 2.45 -> 0.00 mm
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- added copper zone on B.Cu, net +5V
- added copper zone on F.Cu, net +5V
- added copper zone on B.Cu, net +BATT
- added copper zone on F.Cu, net +BATT
- added copper zone on B.Cu, net Net-(J2-Pin_1)
- added copper zone on B.Cu, net Net-(J4-Pin_1)
- added copper zone on B.Cu, net Net-(J4-Pin_2)
- removed copper zone on F.Cu, net Net-(J2-Pin_1)
- removed copper zone on F.Cu, net Net-(J2-Pin_2)
- removed copper zone on F.Cu, net Net-(J4-Pin_1)
- removed copper zone on F.Cu, net Net-(J4-Pin_2)
- removed copper zone on F.Cu, net VCC
Other:
- board size 80 x 36.6 mm -> 80 x 36.5 mm
- board text added: "M_DER"
- board text added: "M_IZ"
